File: ADAFRUIT_LCD_ILI9341.kicad_sch (KiCad schematic)
At the start: 1 part, among them U11 ADAFRUIT2478

Commit message: commit a sound version
Parts:
- added C56: 22u, Capacitor_SMD:C_0805_2012Metric, symbol Device:C
- added C57: 100n, Capacitor_SMD:C_0402_1005Metric, symbol Device:C
Connections:
- net GND: now also C57.2
- net at U11.22 (VIN2): now also C56.2
- net ILI9341_CLK: now reaches U11.24 (CLK)
- net ILI9341_MISO: now reaches U11.25 (MISO)
- net ILI9341_MOSI: now reaches U11.26 (MOSI)
- net ILI9341_CS: now reaches U11.27 (CS2)
- net ILI9341_DC: now reaches U11.28 (D/C)
- new net +3.3V: C56.1, C57.1
- no-connect marks 8 -> 32
