File: BluetoothWifi.kicad_sch (KiCad schematic)
At the start: 6 parts, among them J3 Conn_02x05_Odd_Even, U14 ESP32-WROOM-32D

Commit message: started the layout
Parts:
- R37: footprint Capacitor_SMD:C_0805_2012Metric -> Resistor_SMD:R_0402_1005Metric
Changed lines of the file:
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@@
 			)
 		)
-		(property "Footprint" "Capacitor_SMD:C_0805_2012Metric"
+		(property "Footprint" "Resistor_SMD:R_0402_1005Metric"
 			(at 66.802 68.58 90)
 			(effects
