File: MCU.kicad_sch (KiCad schematic)
At the start: 26 parts, among them U4 STM32H750IBKx

Commit message: Add the SDRAM ic
16MB SDRAM add
Parts:
- removed U4: STM32H750IBKx, UniversalRemoteControllerLibrary:BGA201C65P15X15_1000X1000X60, symbol MCU_ST_STM32H7:STM32H750IBKx
- added U9: STM32H750ZBTx, Package_QFP:LQFP-144_20x20mm_P0.5mm, symbol MCU_ST_STM32H7:STM32H750ZBTx
Connections:
- net +3.3V: now also U9.108 (VDD), U9.121 (VDD), U9.131 (VDD), U9.144 (VDD), U9.17 (VDD), U9.30 (VDD), U9.32 (VREF+), U9.33 (VDDA), U9.39 (VDD), U9.52 (VDD), U9.62 (VDD), U9.72 (VDD), U9.84 (VDD), U9.95 (VDD33_USB)
- net GND: now also U9.107 (VSS), U9.120 (VSS), U9.130 (VSS), U9.143 (PDR_ON), U9.16 (VSS), U9.31 (VSSA), U9.38 (VSS), U9.51 (VSS), U9.61 (VSS), U9.83 (VSS), U9.94 (VSS)
- net at C15.2: now also U9.71 (VCAP)
- net at R14.2: now also U9.138 (BOOT0)
- net at C16.2: now also U9.106 (VCAP)
- net at C13.1, R13.2: now also U9.25 (NRST)
- new net FMC_A0: U9.10 (PF0)
- new net FMC_A1: U9.11 (PF1)
- new net FMC_A10: U9.56 (PG0)
- new net FMC_A11: U9.57 (PG1)
- new net FMC_A2: U9.12 (PF2)
- new net FMC_A3: U9.13 (PF3)
- new net FMC_A4: U9.14 (PF4)
- new net FMC_A5: U9.15 (PF5)
- new net FMC_A6: U9.50 (PF12)
- new net FMC_A7: U9.53 (PF13)
- new net FMC_A8: U9.54 (PF14)
- new net FMC_A9: U9.55 (PF15)
- new net FMC_BA0: U9.89 (PG4)
- new net FMC_BA1: U9.90 (PG5)
- new net FMC_DQ0: U9.85 (PD14)
- new net FMC_DQ1: U9.86 (PD15)
- new net FMC_DQ10: U9.66 (PE13)
- new net FMC_DQ11: U9.67 (PE14)
- new net FMC_DQ12: U9.68 (PE15)
- new net FMC_DQ13: U9.77 (PD8)
- new net FMC_DQ14: U9.78 (PD9)
- new net FMC_DQ15: U9.79 (PD10)
- new net FMC_DQ2: U9.114 (PD0)
- new net FMC_DQ3: U9.115 (PD1)
- new net FMC_DQ4: U9.58 (PE7)
- new net FMC_DQ5: U9.59 (PE8)
- new net FMC_DQ6: U9.60 (PE9)
- new net FMC_DQ7: U9.63 (PE10)
- new net FMC_DQ8: U9.64 (PE11)
- new net FMC_DQ9: U9.65 (PE12)
- new net FMC_NBL0: U9.141 (PE0)
- new net FMC_NBL1: U9.142 (PE1)
- new net FMC_SDCKE: U9.29 (PC3_C)
- new net FMC_SDCLK: U9.93 (PG8)
- new net FMC_SDNCAS: U9.132 (PG15)
- new net FMC_SDNE0: U9.28 (PC2_C)
- new net FMC_SDNRAS: U9.49 (PF11)
- new net FMC_SDNWE: U9.26 (PC0)
- new net QUADSPI_BK1_IO0: U9.20 (PF8)
- new net QUADSPI_BK1_IO1: U9.21 (PF9)
- new net QUADSPI_BK1_IO2: U9.1 (PE2)
- new net QUADSPI_BK1_IO3: U9.18 (PF6)
- new net QUADSPI_BK1_NCS: U9.69 (PB10)
- new net QUADSPI_CLK: U9.22 (PF10)
- new net USB+: U9.104 (PA12)
- new net USB-: U9.103 (PA11)
Other:
- moved on the sheet: C15, C16

Commit message: Add the nrf and joystic module
Parts:
- removed C28, C29: 100n, Capacitor_SMD:C_0402_1005Metric, symbol Device:C
Connections:
- net DEBUG_SWDIO: now reaches U9.105 (PA13)
- net DEBUG_SWDCLK: now reaches U9.109 (PA14)
- net BATT_FET_FLAG: now reaches U9.133 (PB3)
- net ~{BQ25620_INT}: now reaches U9.134 (PB4)
- net ~{BQ25620_CE}: now reaches U9.135 (PB5)
- net I2C_SCK: now reaches U9.136 (PB6)
- net I2C_SDA: now reaches U9.137 (PB7)

Commit message: commit a sound version
Parts:
- added C58, C59: 20p, Capacitor_SMD:C_0402_1005Metric, symbol Device:C
- added J4: Conn_02x07_Odd_Even, UniversalRemoteControllerLibrary:PinHeader_2x07_P1.27mm_Vertical_SMD, symbol UniversalRemoteControllerLibary:Conn_02x07_Odd_Even
- added Y2: FL2500279Z, UniversalRemoteControllerLibrary:FL2500279Z, symbol UniversalRemoteControllerLibary:FL2500279Z
- C35, C36, C37, C38: footprint Capacitor_SMD:C_0805_2012Metric -> Capacitor_SMD:C_0603_1608Metric
Connections:
- net +3.3V: now also J4.3 (Pin_3)
- net BATT_FET_FLAG: now also U9.139 (PB8); no longer U9.133 (PB3)
- net DEBUG_SWDCLK: now also J4.6 (Pin_6), J4.9 (Pin_9)
- net DEBUG_SWDIO: now also J4.4 (Pin_4)
- net GND: now also C58.2, C59.2, J4.11 (Pin_11), J4.5 (Pin_5), J4.7 (Pin_7)
- net ESP32_RX: now reaches U9.101 (PA9)
- net ESP32_TX: now reaches U9.102 (PA10)
- net T_JTDI: now reaches U9.110 (PA15)
- net T_JTDI: now also J4.10 (Pin_10)
- net AXL_SCK: now reaches U9.111 (PC10)
- net AXL_MISO: now reaches U9.112 (PC11)
- net AXL_MOSI: now reaches U9.113 (PC12)
- net ESP32_EN: now reaches U9.119 (PD5)
- net JOY_LEFT_BUTTON: now reaches U9.128 (PG13)
- net JOY_RIGHT_BUTTON: now reaches U9.129 (PG14)
- net XTAL1: now reaches U9.23 (PH0)
- net XTAL1: now also C58.1, Y2.1 (XTAL_1)
- net XTAL2: now reaches U9.24 (PH1)
- net XTAL2: now also C59.1, Y2.3 (XTAL_2)
- net NRST: now reaches C13.1, R13.2, U9.25 (NRST)
- net NRST: now also J4.12 (Pin_12)
- net JOY_LEFT_H_ANALOG: now reaches U9.34 (PA0)
- net JOY_LEFT_V_ANALOG: now reaches U9.35 (PA1)
- net JOY_RIGHT_H_ANALOG: now reaches U9.36 (PA2)
- net JOY_RIGHT_V_ANALOG: now reaches U9.37 (PA3)
- net AXL_INT1: now reaches U9.44 (PC4)
- net AXL_INT2: now reaches U9.45 (PC5)
- net AXL_CS: now reaches U9.7 (PC13)
- net ILI9341_CLK: now reaches U9.70 (PB11)
- net ILI9341_MISO: now reaches U9.73 (PB12)
- net ILI9341_MOSI: now reaches U9.74 (PB13)
- net ILI9341_CS: now reaches U9.75 (PB14)
- net ILI9341_DC: now reaches U9.76 (PB15)
- net BME280_SCK: now reaches U9.81 (PD12)
- net BME280_SDA: now reaches U9.82 (PD13)
- net T_VCP_RX: now reaches U9.96 (PC6)
- net T_VCP_RX: now also J4.13 (Pin_13)
- net T_VCP_TX: now reaches U9.97 (PC7)
- net T_VCP_TX: now also J4.14 (Pin_14)
- new net DEBUG_SWO: J4.8 (Pin_8), U9.133 (PB3)
- no-connect marks 1 -> 3
Other:
- moved on the sheet: C13, R13, R14

Commit message: started the layout
Connections:
- net DEBUG_SWDCLK: no longer J4.9 (Pin_9)
- net I2S_SDO: now reaches U9.123 (PD7)
- net I2S_CLK: now reaches U9.41 (PA5)
- net I2S_SDI: now reaches U9.42 (PA6)
- net SD_MODE_LEFT: now reaches U9.46 (PB0)
- net SD_MODE_RIGHT: now reaches U9.47 (PB1)
- net T_JTDI: no longer names the net of J4.10 (Pin_10)
- net T_JTDI: no longer U9.110 (PA15)
- new net I2C_WS: U9.110 (PA15)
- no-connect marks 3 -> 5
