File: Power.kicad_sch (KiCad schematic)
At the start: 65 parts, among them J1 USB_C_Receptacle_USB2.0_16P, J2 Conn_01x03_Pin, U1 USBLC6-2SC6, U2 TPS631000DRLR, U3 BQ25620RYKR, U5 MAX16054AZT, U6 AP2161W

Commit message: Add the SDRAM ic
16MB SDRAM add
Changed lines of the file:
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@@
 		(on_board yes)
 		(dnp no)
-		(fields_autoplaced yes)
 		(property "Reference" "U3"
-			(at 224.79 184.15 0)
+			(at 216.662 192.278 0)
 			(effects
 				(font
@@
 		)
 		(property "Value" "BQ25620RYKR"
-			(at 224.79 186.69 0)
+			(at 223.52 244.348 0)
 			(effects
 				(font
@@
 					(size 1.27 1.27)
 				)
+				(hide yes)
 			)
 		)
@@
 					(size 1.27 1.27)
 				)
+				(hide yes)
 			)
 		)

Commit message: started the layout
Parts:
- removed C33: 120u, Capacitor_SMD:C_0805_2012Metric, symbol Device:C_Polarized
- added C33: 100u, Capacitor_SMD:C_1206_3216Metric, symbol Device:C
- added C72: 100n, Capacitor_SMD:C_0402_1005Metric, symbol Device:C
- C3: footprint Capacitor_SMD:C_0603_1608Metric -> Capacitor_SMD:C_1206_3216Metric; symbol Device:C_Polarized -> Device:C
- C4: footprint Capacitor_SMD:C_0603_1608Metric -> Capacitor_SMD:C_0805_2012Metric
Connections:
- net +3.3V: now also C72.1
- net GND: now also C33.2, C72.2
- net at C32.1, C4.1, TP2.1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: now also C33.1
Other:
- moved on the sheet: C32, C4
