File: QUADSPI.kicad_sch (KiCad schematic)
At the start: 9 parts, among them U7 W25Q128JVS

Commit message: started the layout
Parts:
- R17: footprint Capacitor_SMD:C_0402_1005Metric -> Resistor_SMD:R_0402_1005Metric
Changed lines of the file:
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@@
 			)
 		)
-		(property "Footprint" "Capacitor_SMD:C_0402_1005Metric"
+		(property "Footprint" "Resistor_SMD:R_0402_1005Metric"
 			(at 138.43 80.518 90)
 			(effects
