File: Sensors.kicad_sch (KiCad schematic)
At the start: 5 parts, among them U10 LSM6DSVTR, U12 JOYSTIC-09032, U13 JOYSTIC-09032, U4 BME280

Commit message: commit a sound version
Parts:
- removed MK1: IM69D130, Sensor_Audio:Infineon_PG-LLGA-5-1, symbol Sensor_Audio:IM69D130
- added C60, C61, C62, C63, C64, C65, C66, C67: 100n, Capacitor_SMD:C_0402_1005Metric, symbol Device:C
- added MK1, MK2: IM69D130, UniversalRemoteControllerLibrary:Infineon_PG-LLGA-5-1, symbol UniversalRemoteControllerLibary:IM69D130
- added R38, R39, R40, R41: 10k, Capacitor_SMD:C_0402_1005Metric, symbol Device:R
- added R42, R43: 4,7k, Capacitor_SMD:C_0402_1005Metric, symbol Device:R
Connections:
- net GND: now also U12.H3 (H-), U12.S1 (SHIELD), U12.S2 (SHIELD), U12.S3 (SHIELD), U12.S4 (SHIELD), U12.V3 (V-), U13.H3 (H-), U13.S1 (SHIELD), U13.S2 (SHIELD), U13.S3 (SHIELD), U13.S4 (SHIELD), U13.V3 (V-), C60.2, C61.2, C62.2, C63.2, C64.2, C65.2, C66.2, C67.2, MK1.5 (GND), MK2.4 (SELECT), MK2.5 (GND), R38.2, R40.2
- net AXL_MISO: now reaches U10.1 (SDO/SA0)
- net AXL_CS: now reaches U10.12 (CS)
- net AXL_SCK: now reaches U10.13 (SCL)
- net AXL_MOSI: now reaches U10.14 (SDA)
- net AXL_INT1: now reaches U10.4 (INT1)
- net +3.3V: now reaches U10.5 (VDDIO)
- net +3.3V: now also U10.8 (VDD), U12.B1A (SEL+), U12.H1 (H+), U12.V1 (V+), U13.B1A (SEL+), U13.H1 (H+), U13.V1 (V+), U4.2 (CSB), U4.6 (VDDIO), U4.8 (VDD), C60.1, C61.1, C64.1, C65.1, C66.1, C67.1, MK1.2 (VDD), MK1.4 (SELECT), MK2.2 (VDD), R42.1, R43.1
- net AXL_INT2: now reaches U10.9 (INT2)
- net at U12.B2A (SEL-): now also R38.1, R39.1
- net JOY_LEFT_H_ANALOG: now reaches U12.H2 (H)
- net JOY_LEFT_V_ANALOG: now reaches U12.V2 (V)
- net BME280_SCK: now reaches U4.4 (SCK)
- net BME280_SCK: now also R43.2
- net BME280_SDA: now reaches U4.5 (SDO)
- net BME280_SDA: now also R42.2
- net at U13.B2A (SEL-): now also R40.1, R41.1
- net JOY_RIGHT_H_ANALOG: now reaches U13.H2 (H)
- net JOY_RIGHT_V_ANALOG: now reaches U13.V2 (V)
- new net JOY_LEFT_BUTTON: C62.1, R39.2
- new net JOY_RIGHT_BUTTON: C63.1, R41.2
- new net MIC_I2S_CLK: MK1.3 (CLOCK), MK2.3 (CLOCK)
- new net MIC_I2S_DATA: MK1.1 (DATA), MK2.1 (DATA)
- no-connect marks 0 -> 5
Other:
- moved on the sheet: U10, U4

Commit message: started the layout
Parts:
- added R44: 10k, Resistor_SMD:R_0402_1005Metric, symbol Device:R
- MK1, MK2: Distributor (none) -> Mouser; OrderCode (none) -> 726-IM69D130V01XTSA1
Connections:
- net +3.3V: now also R44.1; no longer MK1.4 (SELECT)
- net MIC_I2S_CLK renamed I2S_CLK
- net MIC_I2S_DATA renamed I2S_SDI
- new net: MK1.4 (SELECT), R44.2
Other:
- note added: "Left Channel"
- note added: "Right Channel"
Changed lines of the file:
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@@
 		)
 	)
+	(wire
+		(pts
+			(xy 59.69 91.44) (xy 53.34 91.44)
+		)
+		(stroke
+			(width 0)
+			(type default)
+		)
+	)
 	(bus
 		(pts
@@
 	(wire
 		(pts
-			(xy 69.85 91.44) (xy 53.34 91.44)
+			(xy 69.85 91.44) (xy 67.31 91.44)
 		)
 		(stroke
@@
 		)
 	)
-	(label "MIC_I2S_CLK"
+	(text "Right Channel"
+		(exclude_from_sim no)
+		(at 253.492 90.678 0)
+		(effects
+			(font
+				(face "KiCad Font")
+				(size 2.54 2.54)
+				(thickness 0.508)
+				(bold yes)
+			)
+		)
+	)
+	(text "Left Channel"
+		(exclude_from_sim no)
+		(at 87.376 91.694 0)
+		(effects
+			(font
+				(face "KiCad Font")
+				(size 2.54 2.54)
+				(thickness 0.508)
+				(bold yes)
+			)
+		)
+	)
+	(label "I2S_CLK"
 		(at 242.57 99.06 0)
 		(fields_autoplaced yes)
@@
 		)
 	)
-	(label "MIC_I2S_DATA"
+	(label "I2S_SDI"
 		(at 99.06 76.2 0)
 		(fields_autoplaced yes)
@@
 		)
 	)
-	(label "MIC_I2S_DATA"
+	(label "I2S_SDI"
 		(at 242.57 101.6 0)
 		(fields_autoplaced yes)
@@
 		)
 	)
-	(label "MIC_I2S_CLK"
+	(label "I2S_CLK"
 		(at 73.66 101.6 0)
 		(fields_autoplaced yes)
@@
 		)
 	)
-	(label "MIC_I2S_CLK"
+	(label "I2S_CLK"
 		(at 99.06 73.66 0)
 		(fields_autoplaced yes)
@@
 		)
 	)
-	(label "MIC_I2S_DATA"
+	(label "I2S_SDI"
 		(at 73.66 104.14 0)
 		(fields_autoplaced yes)
@@
 		)
 	)
-	(hierarchical_label "MIC_I2S"
+	(hierarchical_label "AUDIO_I2S"
 		(shape bidirectional)
 		(at 157.48 83.82 0)
@@
 			)
 		)
+		(property "OrderCode" "726-IM69D130V01XTSA1"
+			(at 53.34 101.6 0)
+			(effects
+				(font
+					(size 1.27 1.27)
+				)
+				(hide yes)
+			)
+		)
+		(property "Distributor" "Mouser"
+			(at 53.34 101.6 0)
+			(effects
+				(font
+					(size 1.27 1.27)
+				)
+				(hide yes)
+			)
+		)
 		(pin "2"
 		)
@@
 			)
 		)
+		(property "OrderCode" "726-IM69D130V01XTSA1"
+			(at 226.06 99.06 0)
+			(effects
+				(font
+					(size 1.27 1.27)
+				)
+				(hide yes)
+			)
+		)
+		(property "Distributor" "Mouser"
+			(at 226.06 99.06 0)
+			(effects
+				(font
+					(size 1.27 1.27)
+				)
+				(hide yes)
+			)
+		)
 		(pin "2"
 		)
@@
 					(unit 1)
 				)
+			)
+		)
+	)
+	(symbol
+		(lib_id "Device:R")
+		(at 63.5 91.44 90)
+		(unit 1)
+		(exclude_from_sim no)
+		(in_bom yes)
+		(on_board yes)
+		(dnp no)
+		(property "Reference" "R44"
+			(at 63.5 89.154 90)
+			(effects
+				(font
+					(size 1.27 1.27)
+				)
+			)
+		)
+		(property "Value" "10k"
+			(at 63.246 94.234 90)
+			(effects
+				(font
+					(size 1.27 1.27)
+				)
+			)
+		)
+		(property "Footprint" "Resistor_SMD:R_0402_1005Metric"
+			(at 63.5 93.218 90)
+			(effects
+				(font
+					(size 1.27 1.27)
+				)
+				(hide yes)
+			)
+		)
+		(property "Datasheet" "~"
+			(at 63.5 91.44 0)
+			(effects
+				(font
+					(size 1.27 1.27)
+				)
+				(hide yes)
+			)
+		)
+		(property "Description" "Resistor"
+			(at 63.5 91.44 0)
+			(effects
+				(font
+					(size 1.27 1.27)
+				)
+				(hide yes)
+			)
+		)
+		(pin "1"
+		)
+		(pin "2"
+		)
+		(instances
+			(project "UniversalRemoteController"
+				(path "/dfe540b7-7587-4b82-94ea-0a8290455e48/983f520b-4c15-4e26-8d0a-f1f7c260b573"
+					(reference "R44")
+					(unit 1)
+				)
