File: UniversalRemoteController.kicad_pcb (KiCad board)
At the start: 8 copper layers, 141 parts, among them J1 USB_C_Receptacle_USB2.0_16P, J2 Conn_01x03_Pin, U1 USBLC6-2SC6, U10 LSM6DSVTR, U11 ADAFRUIT2478, U12 JOYSTIC-09032, U13 JOYSTIC-09032, U2 TPS631000DRLR, U3 BQ25620RYKR, U4 BME280, U5 MAX16054AZT, U6 AP2161W, U7 W25Q128JVS, U8 IS42S32400F-6TLI, U9 STM32H750ZBTx

Commit message: commit a sound version
Parts:
- added C28: 22u, Capacitor_SMD:C_0805_2012Metric, F.Cu at (217.1, 38.0)
- added C29: 100n, Capacitor_SMD:C_0402_1005Metric, F.Cu at (220.8, 37.5)
- added C55: 100n, Capacitor_SMD:C_0402_1005Metric, F.Cu at (220.8, 39.5)
- added C56: 22u, Capacitor_SMD:C_0805_2012Metric, F.Cu at (158.5, 119.2)
- added C57: 100n, Capacitor_SMD:C_0402_1005Metric, F.Cu at (157.7, 121.7)
- added C58: 20p, Capacitor_SMD:C_0402_1005Metric, F.Cu at (55.0, 49.3)
- added C59: 20p, Capacitor_SMD:C_0402_1005Metric, F.Cu at (55.0, 51.3)
- added C60: 100n, Capacitor_SMD:C_0402_1005Metric, F.Cu at (40.6, 49.3)
- added C61: 100n, Capacitor_SMD:C_0402_1005Metric, F.Cu at (40.6, 51.3)
- added C62: 100n, Capacitor_SMD:C_0402_1005Metric, F.Cu at (40.6, 53.3)
- added C63: 100n, Capacitor_SMD:C_0402_1005Metric, F.Cu at (40.6, 55.2)
- added C64: 100n, Capacitor_SMD:C_0402_1005Metric, F.Cu at (40.6, 57.2)
- added C65: 100n, Capacitor_SMD:C_0402_1005Metric, F.Cu at (43.4, 49.3)
- added C66: 100n, Capacitor_SMD:C_0402_1005Metric, F.Cu at (43.4, 51.3)
- added C67: 100n, Capacitor_SMD:C_0402_1005Metric, F.Cu at (43.4, 53.3)
- added J3: Conn_02x05_Odd_Even, UniversalRemoteControllerLibrary:PinHeader_2x05_P1.27mm_Vertical_SMD, F.Cu at (148.7, 134.9)
- added J3: Conn_02x03_Top_Bottom, Connector_PinHeader_1.00mm:PinHeader_2x03_P1.00mm_Vertical_SMD, F.Cu at (219.1, 34.0)
- added J4: Conn_02x07_Odd_Even, UniversalRemoteControllerLibrary:PinHeader_2x07_P1.27mm_Vertical_SMD, F.Cu at (148.7, 123.2)
- added MK1: IM69D130, UniversalRemoteControllerLibrary:Infineon_PG-LLGA-5-1, F.Cu at (159.0, 133.1)
- added MK2: IM69D130, UniversalRemoteControllerLibrary:Infineon_PG-LLGA-5-1, F.Cu at (42.1, 60.6)
- added R37: 10k, Capacitor_SMD:C_0805_2012Metric, F.Cu at (217.1, 41.0)
- added R38: 10k, Capacitor_SMD:C_0402_1005Metric, F.Cu at (152.2, 88.2)
- added R39: 10k, Capacitor_SMD:C_0402_1005Metric, F.Cu at (152.2, 87.0)
- added R40: 10k, Capacitor_SMD:C_0402_1005Metric, F.Cu at (189.4, 57.4)
- added R41: 10k, Capacitor_SMD:C_0402_1005Metric, F.Cu at (189.4, 60.4)
- added R42: 4,7k, Capacitor_SMD:C_0402_1005Metric, F.Cu at (43.4, 55.2)
- added R43: 4,7k, Capacitor_SMD:C_0402_1005Metric, F.Cu at (43.4, 57.2)
- added U14: ESP32-WROOM-32D, UniversalRemoteControllerLibrary:MODULE_ESP32-WROOM-32D, F.Cu at (218.0, 72.4)
- added U15: MAX98357AEWL+T, UniversalRemoteControllerLibrary:BGA9C40P3X3_144X135X69, F.Cu at (49.1, 58.5)
- added U16: MAX98357AEWL+T, UniversalRemoteControllerLibrary:BGA9C40P3X3_144X135X69, F.Cu at (49.1, 62.9)
- added Y2: FL2500279Z, UniversalRemoteControllerLibrary:FL2500279Z, F.Cu at (50.2, 51.3)
- moved U13 73.4 mm to (270.8, 94.2)
- moved U8 48.4 mm to (105.2, 114.8)
- moved U12 42.7 mm to (169.1, 94.8)
Connections:
- net Net-(U9-NRST) renamed /MCU/NRST
- U10 pad 1: unconnected-(U10-SDO/SA0-Pad1) -> /Sensors/AXL_MISO
- U10 pad 12: unconnected-(U10-CS-Pad12) -> /Sensors/AXL_CS
- U10 pad 13: unconnected-(U10-SCL-Pad13) -> /Sensors/AXL_SCK
- U10 pad 14: unconnected-(U10-SDA-Pad14) -> /Sensors/AXL_MOSI
- U10 pad 4: unconnected-(U10-INT1-Pad4) -> /Sensors/AXL_INT1
- U10 pad 5: unconnected-(U10-VDDIO-Pad5) -> +3.3V
- U10 pad 8: unconnected-(U10-VDD-Pad8) -> +3.3V
- U10 pad 9: unconnected-(U10-INT2-Pad9) -> /Sensors/AXL_INT2
- U11 pad 22: unconnected-(U11-VIN2-Pad22) -> Net-(U11-VIN2)
- U11 pad 24: unconnected-(U11-CLK-Pad24) -> /ADAFRUIT_LCD_ILI9341/ILI9341_CLK
- U11 pad 25: unconnected-(U11-MISO-Pad25) -> /ADAFRUIT_LCD_ILI9341/ILI9341_MISO
- U11 pad 26: unconnected-(U11-MOSI-Pad26) -> /ADAFRUIT_LCD_ILI9341/ILI9341_MOSI
- U11 pad 27: unconnected-(U11-CS2-Pad27) -> /ADAFRUIT_LCD_ILI9341/ILI9341_CS
- U11 pad 28: unconnected-(U11-D/C-Pad28) -> /ADAFRUIT_LCD_ILI9341/ILI9341_DC
- U12 pad B1A: unconnected-(U12-SEL+-PadB1A) -> +3.3V
- U12 pad B2A: unconnected-(U12-SEL--PadB2A) -> Net-(U12-SEL-)
- U12 pad H1: unconnected-(U12-H+-PadH1) -> +3.3V
- U12 pad H2: unconnected-(U12-H-PadH2) -> /MCU/JOY_LEFT_H_ANALOG
- U12 pad H3: unconnected-(U12-H--PadH3) -> GND
- U12 pad S1: Net-(U12-SHIELD-PadS1) -> GND
- U12 pad S2: Net-(U12-SHIELD-PadS1) -> GND
- U12 pad S3: Net-(U12-SHIELD-PadS1) -> GND
- U12 pad S4: Net-(U12-SHIELD-PadS1) -> GND
- U12 pad V1: unconnected-(U12-V+-PadV1) -> +3.3V
- U12 pad V2: unconnected-(U12-V-PadV2) -> /MCU/JOY_LEFT_V_ANALOG
- U12 pad V3: unconnected-(U12-V--PadV3) -> GND
- U13 pad B1A: unconnected-(U13-SEL+-PadB1A) -> +3.3V
- U13 pad B2A: unconnected-(U13-SEL--PadB2A) -> Net-(U13-SEL-)
- U13 pad H1: unconnected-(U13-H+-PadH1) -> +3.3V
- U13 pad H2: unconnected-(U13-H-PadH2) -> /MCU/JOY_RIGHT_H_ANALOG
- U13 pad H3: unconnected-(U13-H--PadH3) -> GND
- U13 pad S1: Net-(U13-SHIELD-PadS1) -> GND
- U13 pad S2: Net-(U13-SHIELD-PadS1) -> GND
- U13 pad S3: Net-(U13-SHIELD-PadS1) -> GND
- U13 pad S4: Net-(U13-SHIELD-PadS1) -> GND
- U13 pad V1: unconnected-(U13-V+-PadV1) -> +3.3V
- U13 pad V2: unconnected-(U13-V-PadV2) -> /MCU/JOY_RIGHT_V_ANALOG
- U13 pad V3: unconnected-(U13-V--PadV3) -> GND
- U4 pad 2: unconnected-(U4-CSB-Pad2) -> +3.3V
- U4 pad 4: unconnected-(U4-SCK-Pad4) -> /Sensors/BME280_SCK
- U4 pad 5: unconnected-(U4-SDO-Pad5) -> /Sensors/BME280_SDA
- U4 pad 6: unconnected-(U4-VDDIO-Pad6) -> +3.3V
- U4 pad 8: unconnected-(U4-VDD-Pad8) -> +3.3V
- U9 pad 100: unconnected-(U9-PA8-Pad100) -> /MCU/MIC_I2S_CLK
- U9 pad 101: unconnected-(U9-PA9-Pad101) -> /BluetoothWiFi/ESP32_RX
- U9 pad 102: unconnected-(U9-PA10-Pad102) -> /BluetoothWiFi/ESP32_TX
- U9 pad 105: unconnected-(U9-PA13-Pad105) -> /MCU/DEBUG_SWDIO
- U9 pad 109: unconnected-(U9-PA14-Pad109) -> /MCU/DEBUG_SWDCLK
- U9 pad 110: unconnected-(U9-PA15-Pad110) -> /MCU/T_JTDI
- U9 pad 111: unconnected-(U9-PC10-Pad111) -> /MCU/AXL_SCK
- U9 pad 112: unconnected-(U9-PC11-Pad112) -> /MCU/AXL_MISO
- U9 pad 113: unconnected-(U9-PC12-Pad113) -> /MCU/AXL_MOSI
- U9 pad 119: unconnected-(U9-PD5-Pad119) -> /BluetoothWiFi/ESP32_EN
- U9 pad 128: unconnected-(U9-PG13-Pad128) -> /MCU/JOY_LEFT_BUTTON
- U9 pad 129: unconnected-(U9-PG14-Pad129) -> /MCU/JOY_RIGHT_BUTTON
- U9 pad 133: /MCU/BATT_FET_FLAG -> /MCU/DEBUG_SWO
- U9 pad 139: unconnected-(U9-PB8-Pad139) -> /MCU/BATT_FET_FLAG
- U9 pad 23: unconnected-(U9-PH0-Pad23) -> /MCU/XTAL1
- U9 pad 24: unconnected-(U9-PH1-Pad24) -> /MCU/XTAL2
- U9 pad 34: unconnected-(U9-PA0-Pad34) -> /MCU/JOY_LEFT_H_ANALOG
- U9 pad 35: unconnected-(U9-PA1-Pad35) -> /MCU/JOY_LEFT_V_ANALOG
- U9 pad 36: unconnected-(U9-PA2-Pad36) -> /MCU/JOY_RIGHT_H_ANALOG
- U9 pad 37: unconnected-(U9-PA3-Pad37) -> /MCU/JOY_RIGHT_V_ANALOG
- U9 pad 44: unconnected-(U9-PC4-Pad44) -> /MCU/AXL_INT1
- U9 pad 45: unconnected-(U9-PC5-Pad45) -> /MCU/AXL_INT2
- U9 pad 7: unconnected-(U9-PC13-Pad7) -> /MCU/AXL_CS
- U9 pad 70: unconnected-(U9-PB11-Pad70) -> /MCU/ILI9341_CLK
- U9 pad 73: unconnected-(U9-PB12-Pad73) -> /MCU/ILI9341_MISO
- U9 pad 74: unconnected-(U9-PB13-Pad74) -> /MCU/ILI9341_MOSI
- U9 pad 75: unconnected-(U9-PB14-Pad75) -> /MCU/ILI9341_CS
- U9 pad 76: unconnected-(U9-PB15-Pad76) -> /MCU/ILI9341_DC
- U9 pad 81: unconnected-(U9-PD12-Pad81) -> /MCU/BME280_SCK
- U9 pad 82: unconnected-(U9-PD13-Pad82) -> /MCU/BME280_SDA
- U9 pad 96: unconnected-(U9-PC6-Pad96) -> /MCU/T_VCP_RX
- U9 pad 97: unconnected-(U9-PC7-Pad97) -> /MCU/T_VCP_TX
- U9 pad 99: unconnected-(U9-PC9-Pad99) -> /MCU/MIC_I2S_DATA

Commit message: started the layout
Parts:
- removed the C28 at (217.1, 38.0)
- removed the C28 at (135.2, 66.4)
- removed the C29 at (220.8, 37.5)
- removed the C29 at (135.2, 68.3)
- removed the J3 at (148.7, 134.9)
- removed the J3 at (219.1, 34.0)
- removed the MK1 at (159.0, 133.1)
- removed the MK1 at (212.1, 125.5)
- removed the R14 at (152.9, 64.7)
- removed the R14 at (195.8, 85.5)
- added C28: 22u, Capacitor_SMD:C_0805_2012Metric, F.Cu at (236.1, 43.3)
- added C29: 100n, Capacitor_SMD:C_0402_1005Metric, F.Cu at (249.3, 18.8)
- added C68: 10u, Capacitor_SMD:C_0805_2012Metric, F.Cu at (44.7, 88.7)
- added C69: 0,1u, Capacitor_SMD:C_0603_1608Metric, F.Cu at (31.0, 92.2)
- added C70: 10u, Capacitor_SMD:C_0805_2012Metric, F.Cu at (44.7, 91.7)
- added C71: 0,1u, Capacitor_SMD:C_0603_1608Metric, F.Cu at (31.0, 94.7)
- added C72: 100n, Capacitor_SMD:C_0402_1005Metric, F.Cu at (177.7, 140.7)
- added J3: Conn_02x05_Odd_Even, UniversalRemoteControllerLibrary:PinHeader_2x05_P1.27mm_Vertical_SMD, F.Cu at (239.3, 37.5)
- added J5: Conn_01x02_Pin, Connector_PinHeader_2.54mm:PinHeader_1x02_P2.54mm_Horizontal, F.Cu at (31.4, 78.9)
- added J6: Conn_01x02_Pin, Connector_PinHeader_2.54mm:PinHeader_1x02_P2.54mm_Horizontal, F.Cu at (31.4, 86.1)
- added MK1: IM69D130, UniversalRemoteControllerLibrary:Infineon_PG-LLGA-5-1, F.Cu at (89.4, 19.1)
- added R14: 10k, Capacitor_SMD:C_0805_2012Metric, F.Cu at (208.7, 43.8)
- added R44: 10k, Resistor_SMD:R_0402_1005Metric, F.Cu at (98.2, 17.6)
- added R45: 210k, Resistor_SMD:R_0402_1005Metric, F.Cu at (34.5, 92.0)
- C3: footprint Capacitor_SMD:C_0603_1608Metric -> Capacitor_SMD:C_1206_3216Metric
- C33: value 120u -> 100u; footprint Capacitor_SMD:C_0805_2012Metric -> Capacitor_SMD:C_1206_3216Metric
- C35, C36, C37, C38: footprint Capacitor_SMD:C_0805_2012Metric -> Capacitor_SMD:C_0603_1608Metric
- C4: footprint Capacitor_SMD:C_0603_1608Metric -> Capacitor_SMD:C_0805_2012Metric
- FL1, J1, J4, U8, U9: moved to B.Cu
- R17: footprint Capacitor_SMD:C_0402_1005Metric -> Resistor_SMD:R_0402_1005Metric
- R37: footprint Capacitor_SMD:C_0805_2012Metric -> Resistor_SMD:R_0402_1005Metric
- U15, U16: value MAX98357AEWL+T -> MAX98357AETE+T; footprint UniversalRemoteControllerLibrary:BGA9C40P3X3_144X135X69 -> UniversalRemoteControllerLibrary:QFN50P300X300X80-17N
- moved R32 171.9 mm to (204.4, 18.4)
- moved R25 164.4 mm to (191.2, 18.1)
- moved R26 164.4 mm to (191.2, 20.1)
- moved R27 164.4 mm to (191.2, 22.0)
- moved R28 164.4 mm to (191.2, 24.0)
- moved R29 164.4 mm to (191.2, 26.0)
- moved R30 164.4 mm to (191.2, 27.9)
- moved R31 164.4 mm to (191.2, 29.9)
- moved R33 164.4 mm to (194.1, 20.1)
- moved R34 164.4 mm to (194.1, 22.0)
- moved R35 164.4 mm to (194.1, 24.0)
- moved R36 164.4 mm to (194.1, 26.0)
- moved C40 164.4 mm to (182.6, 18.1)
- moved C42 164.4 mm to (182.6, 20.1)
- moved C43 164.4 mm to (182.6, 22.0)
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Connections:
- J4 pad 10: /MCU/T_JTDI -> unconnected-(J4-Pin_10-Pad10)
- J4 pad 9: /MCU/DEBUG_SWDCLK -> unconnected-(J4-Pin_9-Pad9)
- MK2 pad 1: /Sensors/MIC_I2S_DATA -> /Sensors/I2S_SDI
- MK2 pad 3: /Sensors/MIC_I2S_CLK -> /Sensors/I2S_CLK
- U9 pad 100: /MCU/MIC_I2S_CLK -> unconnected-(U9-PA8-Pad100)
- U9 pad 110: /MCU/T_JTDI -> /MCU/I2C_WS
- U9 pad 123: unconnected-(U9-PD7-Pad123) -> /MCU/I2S_SDO
- U9 pad 41: unconnected-(U9-PA5-Pad41) -> /MCU/I2S_CLK
- U9 pad 42: unconnected-(U9-PA6-Pad42) -> /MCU/I2S_SDI
- U9 pad 46: unconnected-(U9-PB0-Pad46) -> /MCU/SD_MODE_LEFT
- U9 pad 47: unconnected-(U9-PB1-Pad47) -> /MCU/SD_MODE_RIGHT
- U9 pad 99: /MCU/MIC_I2S_DATA -> unconnected-(U9-PC9-Pad99)
Routing:
- net /MCU/FMC_DQ15: track 0.00 -> 50.4 mm
- net /MCU/FMC_DQ14: track 0.00 -> 50.0 mm
- net /MCU/FMC_DQ13: track 0.00 -> 45.0 mm
- net /MCU/FMC_DQ12: track 0.00 -> 40.5 mm
- net /MCU/QUADSPI_BK1_IO2: track 31.1 -> 0.00 mm
- net /MCU/QUADSPI_BK1_IO1: track 25.5 -> 0.00 mm
- net /Power/VBUS+: track 0.00 -> 13.7 mm, vias 0 -> 2
- net Net-(D1-K): track 0.00 -> 8.31 mm
- net +VSW: track 0.00 -> 7.38 mm
- net /Power/UP_USB_D-: track 0.00 -> 5.52 mm
- net /Power/UP_USB_D+: track 0.00 -> 5.44 mm
- net /MCU/~{BQ25620_CE}: track 0.00 -> 5.28 mm
- net +3.3V: track 0.00 -> 5.08 mm, vias 0 -> 5
- net Net-(C2-Pad1): track 0.00 -> 4.90 mm
- net /MCU/I2C_SDA: track 0.00 -> 4.19 mm
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- added copper zone on F.Cu, net +3.3V
- added copper zone on F.Cu, net GND
- added copper zone on F.Cu, net Net-(U2-EN)
- added copper zone on In2.Cu, net Net-(U3-SW)
Other:
- board outline added: 150 x 86.7 mm
- copper layers 8 -> 6
