File: audio.kicad_sch (KiCad schematic)
At the start: 2 parts, among them U15 MAX98357AETE+T, U16 MAX98357AETE+T

Commit message: started the layout
Parts:
- added C68, C70: 10u, Capacitor_SMD:C_0805_2012Metric, symbol Device:C
- added C69, C71: 0,1u, Capacitor_SMD:C_0603_1608Metric, symbol Device:C
- added J5, J6: Conn_01x02_Pin, Connector_PinHeader_2.54mm:PinHeader_1x02_P2.54mm_Horizontal, symbol Connector:Conn_01x02_Pin
- added R45: 210k, Resistor_SMD:R_0402_1005Metric, symbol Device:R
Connections:
- net GND: now also U15.2 (GAIN_SLOT), U16.11 (GND_2), U16.15 (GND_3), U16.17 (THERMAL_PAD), U16.2 (GAIN_SLOT), U16.3 (GND_1), C68.2, C69.2, C70.2, C71.2
- net I2S_SDO: now reaches U15.1 (DIN)
- net I2S_SDO: now also U16.1 (DIN)
- net at U15.10 (OUTN): now also J5.2 (Pin_2)
- net I2S_WS: now reaches U15.14 (LRCLK)
- net I2S_WS: now also U16.14 (LRCLK)
- net I2S_CLK: now reaches U15.16 (BCLK)
- net I2S_CLK: now also U16.16 (BCLK)
- net SD_MODE_LEFT: now reaches U15.4 (~{SD_MODE})
- net +3.3V: now reaches U15.7 (VDD_1)
- net +3.3V: now also U15.8 (VDD_2), U16.7 (VDD_1), U16.8 (VDD_2), C68.1, C69.1, C70.1, C71.1, R45.2
- net at U15.9 (OUTP): now also J5.1 (Pin_1)
- net at U16.10 (OUTN): now also J6.2 (Pin_2)
- net SD_MODE_RIGHT: now reaches U16.4 (~{SD_MODE})
- net SD_MODE_RIGHT: now also R45.1
- net at U16.9 (OUTP): now also J6.1 (Pin_1)
Other:
- note added: "Left Channel"
- note added: "Right Channel"
- title: (none) -> Audio
- moved on the sheet: U15
